File: 10segment_led.kicad_sch (KiCad schematic)
At the start: 33 parts, among them U10 led_seg_pos_10, U11 led_seg_pos_10, U12 74HC595, U13 led_seg_pos_10, U14 led_seg_pos_10, U15 led_seg_pos_10, U16 led_seg_pos_10, U17 led_seg_pos_10, U18 led_seg_pos_10, U6 led_seg_pos_10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

Commit message: modify packet of res
Parts:
- added R34: 0, Resistor_SMD:R_0603_1608Metric, symbol Device:R
- R13, R14, R15, R16, R17, R18, R19, R20, R21, R22, R23, R24, R25, R26, R27, R28, R29, R30, R31, R32: footprint (none) -> Resistor_SMD:R_0603_1608Metric
- U12, U7, U9: footprint (none) -> Package_SO:SOIC-16_3.9x9.9mm_P1.27mm
Connections:
- net +5V: no longer names the net of U12.10 (~{SRCLR}), U7.10 (~{SRCLR}), U9.10 (~{SRCLR})
- net +5V: now also R34.1; no longer U12.16 (VCC), U7.16 (VCC), U9.16 (VCC)
- new net VCC5V: R34.2, U12.16 (VCC), U7.16 (VCC), U9.16 (VCC)
