File: led_scroll.kicad_sch (KiCad schematic)
At the start: 5 parts, among them J1 KF128_5.08_2P, J2 KF128_5.08_2P, SW1 RotaryEncoder_Switch, U1 AMS1117-5, U2 ESP32-DEVKITC-32D

Commit message: modify packet of res
Parts:
- added U19: AMS1117-5, Power_Module:AMS1117, symbol Power_Module:AMS1117-5
Connections:
- net +9V: now also U19.1 (Vin)
- net GND: now also U19.2 (GND), U19.3 (GND)
- net led_DIO: now also U2.29 (IO5); no longer U2.31 (IO16)
- net led_RCLK: now also U2.31 (IO16); no longer U2.30 (IO17)
- net led_SCLK: now also U2.30 (IO17); no longer U2.29 (IO5)
- net +3.3V: no longer names the net of U2.1 (3V3)
- net +5V renamed VCC5V
- net VCC5V: now also U19.4 (Vout)
- no-connect marks 22 -> 23
Other:
- sheet 10SEGMENT_LED ports: added VCC5V; removed none
- sheet 4BIT_7SEGMENT_LED ports: added VCC5V; removed none
- moved on the sheet: J1, J2, SW1, U1
